Commit message: commit

File: urdf/mbot.xacro (robot description, xacro)
@@ -38,5 +38,5 @@
   		</transmission>
 	</xacro:macro>
-	<xacro:macro name="wheel_link" params="prefix suffix xreflect yreflect">
+	<xacro:macro name="wheel_link" params="prefix suffix xreflect yreflect friction">
 		<link name="wheel_${prefix}_${suffix}">
 			<visual>
@@ -67,16 +67,18 @@
 		</joint>
 		<gazebo reference="wheel_${prefix}_${suffix}">
-			<mu1 value="200.0"/>
-        	<mu2 value="100.0"/>
-        	<kp value="10000000.0" />
-        	<kd value="1.0" />
+			<mu1 value="${friction*100000.0}"/>
+        	<mu2 value="${friction*100000.0}"/>
+        	<!--<kp value="10000000.0"/>-->
+        	<!--<kd value="1.0" />-->
         	<material>Gazebo/Black</material>
 		</gazebo>
 		<xacro:wheel_tran prefix="${prefix}" suffix="${suffix}"/>
 	</xacro:macro>
-	<xacro:wheel_link prefix="front" suffix="left" xreflect="1.0" yreflect="1.0"/>
-	<xacro:wheel_link prefix="front" suffix="right" xreflect="1.0" yreflect="-1.0"/>
-	<xacro:wheel_link prefix="rear" suffix="left" xreflect="-1.0" yreflect="1.0"/>
-	<xacro:wheel_link prefix="rear" suffix="right" xreflect="-1.0" yreflect="-1.0"/>
+	<xacro:wheel_link prefix="front" suffix="left" xreflect="1.0" yreflect="1.0" friction="0"/>
+	<xacro:wheel_link prefix="front" suffix="right" xreflect="1.0" yreflect="-1.0" friction="0"/>
+	<xacro:wheel_link prefix="rear" suffix="left" xreflect="-1.0" yreflect="1.0" friction="0"/>
+	<xacro:wheel_link prefix="rear" suffix="right" xreflect="-1.0" yreflect="-1.0" friction="0"/>
+	<xacro:wheel_link prefix="center" suffix="left" xreflect="0" yreflect="1.0" friction="1.0"/>
+	<xacro:wheel_link prefix="center" suffix="right" xreflect="0" yreflect="-1.0" friction="1.0"/>
     <link name="imu_link">
         <visual>
@@ -119,5 +121,5 @@
 				<xyzOffset>0 0 0</xyzOffset>
 				<rpyOffset>0 0 0</rpyOffset>
-				<frameName>imu</frameName>
+				<frameName>imu_link</frameName>
 			</plugin>
 			<pose>0 0 0 0 0 0</pose>
@@ -193,4 +195,167 @@
 		</sensor>
 	</gazebo>
+	<link name="laser_link">
+		<visual>
+			<origin xyz="0 0 -0.015" rpy="0 0 0"/>
+			<geometry>
+				<box size="0.03 0.03 0.05"/>
+			</geometry>
+			<material name="grey">
+				<color rgba="0.2 0.2 0.2 1"/>
+			</material>
+		</visual>
+		<collision>
+			<origin xyz="0 0 -0.015" rpy="0 0 0"/>
+			<geometry>
+				<box size="0.02 0.02 0.05"/>
+			</geometry>
+		</collision>
+		<inertial>
+			<origin xyz="0 0 0.04" rpy="0 0 0"/>
+			<mass value="0.01"/>
+			<inertia ixx="0.000001" ixy="0.0" ixz="0.0" iyy="0.000001" iyz="0.0" izz="0.0000001"/>
+		</inertial>
+	</link>
+	<joint name="base_to_laser" type="fixed">
+		<axis rpy="0 0 0" xyz="0 0 1"/>
+		<parent link="base_link"/>
+		<child link="laser_link"/>
+		<origin rpy="0 0 0" xyz="0 0 0.09"/>
+	</joint>
+	<gazebo reference="laser_link">
+		<sensor type="gpu_ray" name="head_hokuyo_sensor">
+			<pose>0 0 0 0 0 0</pose>
+			<visualize>0</visualize>
+			<update_rate>40</update_rate>
+			<ray>
+				<scan>
+					<horizontal>
+						<samples>270</samples>
+						<resolution>1</resolution>
+						<min_angle>-2.356194</min_angle>
+						<max_angle>2.356194</max_angle>
+					</horizontal>
+				</scan>
+				<range>
+					<min>0.10</min>
+					<max>30.0</max>
+					<resolution>0.01</resolution>
+				</range>
+				<noise>
+					<type>gaussian</type>
+					<!-- Noise parameters based on published spec for Hokuyo laser
+						 achieving "+-30mm" accuracy at range < 10m.  A mean of 0.0m and
+						 stddev of 0.01m will put 99.7% of samples within 0.03m of the true
+						 reading. -->
+					<mean>0.0</mean>
+					<stddev>0.01</stddev>
+				</noise>
+			</ray>
+			<plugin name="gazebo_ros_head_hokuyo_controller" filename="libgazebo_ros_gpu_laser.so">
+				<topicName>/mbot/laser/scan</topicName>
+				<frameName>laser_link</frameName>
+			</plugin>
+		</sensor>
+  	</gazebo>
+	<link name="pointer_base">
+		<visual>
+			<geometry>
+				<box size="0.01 0.01 0.005"/>
+			</geometry>
+			<material name="blue2">
+				<color rgba="0.0 0.0 0.5 1.0"/>
+			</material>
+		</visual>
+		<collision>
+			<geometry>
+				<box size="0.01 0.01 0.005"/>
+			</geometry>
+		</collision>
+		<inertial>
+			<mass value="0.01"/>
+			<inertia ixx="0.000001" ixy="0.0" ixz="0.0" iyy="0.000001" iyz="0.0" izz="0.0000001"/>
+		</inertial>
+	</link>
+	<joint name="base_to_pointer_mount" type="fixed">
+		<axis rpy="0 0 0" xyz="1 0 0"/>
+		<parent link="base_link"/>
+		<child link="pointer_base"/>
+		<origin rpy="0 0 0" xyz="0.105 0 0"/>
+	</joint>
+	<gazebo reference="pointer_base">
+		<material>Gazebo/Grey</material>
+	</gazebo>
+	<link name="pointer_link">
+		<visual>
+			<geometry>
+				<cylinder length="0.007" radius="0.0005"/>
+			</geometry>
+			<origin xyz="0 0 0" rpy="0 1.57075 0"/>
+			<material name="red">
+				<color rgba="0.6 0 0 1.0"/>
+			</material>
+		</visual>
+		<collision>
+			<geometry>
+				<cylinder length="0.007" radius="0.0005"/>
+			</geometry>
+			<origin xyz="0 0 0" rpy="0 1.57075 0"/>
+		</collision>
+		<inertial>
+			<mass value="0.001"/>
+			<inertia ixx="0.000001" ixy="0.0" ixz="0.0" iyy="0.000001" iyz="0.0" izz="0.0000001"/>
+		</inertial>
+	</link>
+	<gazebo reference="pointer_link">
+		<material>Gazebo/Red</material>
+		<sensor type="gpu_ray" name="pointer">
+			<pose>0 0 0 0 0 0</pose>
+			<visualize>false</visualize>
+			<update_rate>40</update_rate>
+			<ray>
+				<scan>
+					<horizontal>
+						<samples>3</samples>
+						<resolution>1</resolution>
+						<min_angle>-0.017453</min_angle>
+						<max_angle>0.017453</max_angle>
+					</horizontal>
+				</scan>
+				<range>
+					<min>0.10</min>
+					<max>30.0</max>
+					<resolution>0.01</resolution>
+				</range>
+				<noise>
+					<type>gaussian</type>
+					<!-- Noise parameters based on published spec for Hokuyo laser
+						 achieving "+-30mm" accuracy at range < 10m.  A mean of 0.0m and
+						 stddev of 0.01m will put 99.7% of samples within 0.03m of the true
+						 reading. -->
+					<mean>0.0</mean>
+					<stddev>0.01</stddev>
+				</noise>
+			</ray>
+			<plugin name="gazebo_ros_head_hokuyo_controller" filename="libgazebo_ros_gpu_laser.so">
+				<topicName>/mbot/pointer/scan</topicName>
+				<frameName>pinter_link</frameName>
+			</plugin>
+		</sensor>
+	</gazebo>
+	<joint name="mount_to_pointer" type="continuous">
+		<axis rpy="0 0 0" xyz="0 0 1"/>
+		<parent link="pointer_base"/>
+		<child link="pointer_link"/>
+		<origin xyz="0 0 0.003" rpy="0 0 0"/>
+	</joint>
+	<transmission name="pointer_servo">
+		<type>transmission_interface/SimpleTransmission</type>
+		<joint name="mount_to_pointer">
+			<hardwareInterface>hardware_interface/EffortJointInterface</hardwareInterface>
+		</joint>
+		<actuator name="pointer_motor">
+			<mechanicalReduction>1</mechanicalReduction>
+		</actuator>
+	</transmission>
 	<gazebo>
         <plugin name="gazebo_ros_control" filename="libgazebo_ros_control.so">
